File: ArduinoInputExpander_v0.0.sch (KiCad schematic (older format))
At the start: 59 parts

Commit message: stuff
Parts:
- C1, C2: renamed from C?; footprint (none) -> Capacitors_SMD:C_0805
- J1, J2: renamed from J?; footprint (none) -> Pin_Headers:Pin_Header_Straight_2x02_Pitch2.54mm
- J10, J3, J4, J5, J6, J7, J8, J9: renamed from J?; footprint (none) -> Connectors_Terminal_Blocks:TerminalBlock_Pheonix_PT-3.5mm_8pol
- R1, R10, R11, R12, R13, R14, R15, R16, R17, R18, R19, R2, R20, R21, R22, R23, R24, R25, R26, R27, R28, R29, R3, R30, R31, R32, R33, R4, R5, R6, R7, R8, R9: renamed from R?; footprint (none) -> Resistors_SMD:R_0805
- RV1: renamed from RV?; footprint (none) -> Potentiometers:Potentiometer_Trimmer_Bourns_3339P_Horizontal
- U1, U3, U4, U5, U6: renamed from U?; footprint (none) -> SMD_Packages:SO-16-N
- U10, U11, U7, U8, U9: renamed from U?; footprint (none) -> SMD_Packages:SOIC-14_N
- U2: renamed from U?; footprint (none) -> SMD_Packages:SOIC-8-N
- XA1: renamed from XA?; footprint (none) -> libraries:ARDUINOSHIELDMOD
Connections:
- net GND: now also XA1.GND1 (GND), XA1.GND2 (GND), XA1.GND3 (GND)
- net VCC: now also J1.3 (P3), J10.1 (P1), J10.3 (P3), J10.5 (P5), J10.7 (P7), J3.2 (P2), J3.4 (P4), J3.6 (P6), J3.8 (P8), J4.2 (P2), J4.4 (P4), J4.6 (P6), J4.8 (P8), J5.2 (P2), J5.4 (P4), J5.6 (P6), J5.8 (P8), J6.2 (P2), J6.4 (P4), J6.6 (P6), J6.8 (P8), J7.1 (P1), J7.3 (P3), J7.5 (P5), J7.7 (P7), J8.1 (P1), J8.3 (P3), J8.5 (P5), J8.7 (P7), J9.1 (P1), J9.3 (P3), J9.5 (P5), J9.7 (P7), R1.1, U10.14 (VDD), U11.14 (VDD), U2.4 (R), U2.8 (VCC), U3.16 (VCC), U4.16 (VCC), U5.16 (VCC), U6.16 (VCC), U7.14 (VDD), U8.14 (VDD), U9.14 (VDD), XA1.5V1 (5V)
- net at U6.13 (QH), XA1.D3 (D3_INT1): now also U3.1 (SER)
- net at XA1.D5: now also U1.1; no longer U1.4
- net at J4.1 (P1), U3.10 (E), U8.5 (D): now also R6.2
- net at J4.3 (P3), U3.11 (F), U8.4 (C): now also R7.2
- net at J4.5 (P5), U3.12 (G), U8.3 (B): now also R8.2
- net at J4.7 (P7), U3.14 (H), U8.2 (A): now also R9.2
- net at J3.1 (P1), U3.2 (A), U8.12 (H): now also R2.2
- net at J3.3 (P3), U3.3 (B), U8.11 (G): now also R3.2
- net at J3.5 (P5), U3.4 (C), U8.10 (F): now also R4.2
- net at J3.7 (P7), U3.5 (D), U8.9 (E): now also R5.2
- net at U3.7 (CLK), U4.7 (CLK), U5.7 (CLK)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: now also U1.3; no longer U1.6
- net at J6.1 (P1), U4.10 (E), U9.5 (D): now also R14.2
- net at J6.3 (P3), U4.11 (F), U9.4 (C): now also R15.2
- net at J6.5 (P5), U4.12 (G), U9.3 (B): now also R16.2
- net at J6.7 (P7), U4.14 (H), U9.2 (A): now also R17.2
- net at J5.1 (P1), U4.2 (A), U9.12 (H): now also R10.2
- net at J5.3 (P3), U4.3 (B), U9.11 (G): now also R11.2
- net at J5.5 (P5), U4.4 (C), U9.10 (F): now also R12.2
- net at J5.7 (P7), U4.5 (D), U9.9 (E): now also R13.2
- net at J8.2 (P2), U10.5 (D), U5.10 (E): now also R19.1
- net at J8.4 (P4), U10.4 (C), U5.11 (F): now also R23.1
- net at J8.6 (P6), U10.3 (B), U5.12 (G): now also R27.1
- net at J8.8 (P8), U10.2 (A), U5.14 (H): now also R31.1
- net at J7.2 (P2), U10.12 (H), U5.2 (A): now also R18.1
- net at J7.4 (P4), U10.11 (G), U5.3 (B): now also R22.1
- net at J7.6 (P6), U10.10 (F), U5.4 (C): now also R26.1
- net at J7.8 (P8), U10.9 (E), U5.5 (D): now also R30.1
- net at J10.2 (P2), U11.5 (D), U6.10 (E): now also R21.1
- net at J10.4 (P4), U11.4 (C), U6.11 (F): now also R25.1
- net at J10.6 (P6), U11.3 (B), U6.12 (G): now also R29.1
- net at J10.8 (P8), U11.2 (A), U6.14 (H): now also R33.1
- net at J9.2 (P2), U11.12 (H), U6.2 (A): now also R20.1
- net at J9.4 (P4), U11.11 (G), U6.3 (B): now also R24.1
- net at J9.6 (P6), U11.10 (F), U6.4 (C): now also R28.1
- net at J9.8 (P8), U11.9 (E), U6.5 (D): now also R32.1
- net at J2.2 (P2), U7.1 (K-OR): now also U1.5; no longer U1.2
- net at J2.1 (P1), J2.3 (P3): now also U1.4; no longer U1.1
- removed net 5VDC: J1.3 (P3), J10.1 (P1), J10.3 (P3), J10.5 (P5), J10.7 (P7), J3.2 (P2), J3.4 (P4), J3.6 (P6), J3.8 (P8), J4.2 (P2), J4.4 (P4), J4.6 (P6), J4.8 (P8), J5.2 (P2), J5.4 (P4), J5.6 (P6), J5.8 (P8), J6.2 (P2), J6.4 (P4), J6.6 (P6), J6.8 (P8), J7.1 (P1), J7.3 (P3), J7.5 (P5), J7.7 (P7), J8.1 (P1), J8.3 (P3), J8.5 (P5), J8.7 (P7), J9.1 (P1), J9.3 (P3), J9.5 (P5), J9.7 (P7), R1.1, R10.2, R11.2, R12.2, R13.2, R14.2, R15.2, R16.2, R17.2, R18.1, R19.1, R2.2, R20.1, R21.1, R22.1, R23.1, R24.1, R25.1, R26.1, R27.1, R28.1, R29.1, R3.2, R30.1, R31.1, R32.1, R33.1, R4.2, R5.2, R6.2, R7.2, R8.2, R9.2, U10.14 (VDD), U11.14 (VDD), U2.4 (R), U2.8 (VCC), U3.16 (VCC), U4.16 (VCC), U5.16 (VCC), U6.16 (VCC), U7.14 (VDD), U8.14 (VDD), U9.14 (VDD)
- new net: U1.2, U1.6, XA1.D2 (D2_INT0)
- no-connect marks 16 -> 48
